File: usbsniff_v02.sch (KiCad schematic (older format))
At the start: 23 parts, among them P1 CONN_01X02, P2 CONN_01X08, P3 CONN_01X08, U1 AMS1117, U2 MAX3421E, U3 MAX3421E, X1 USB_type_A, X2 micro_USB, Y1 Crystal_Small, Y2 Crystal_Small

Commit message: add LED, redesign pcb
Parts:
- added C10, C12: 1uF, Capacitors_SMD:C_0805, symbol C_Small
- added C11: 10uF, Capacitors_Tantalum_SMD:TantalC_SizeB_EIA-3528_Reflow, symbol CP_Small
- added C13: 0.1uF, Capacitors_SMD:C_0805, symbol C_Small
- added D1, D2: LED, LEDs:LED-3MM, symbol LED
- added R5, R6: 470 Ohm, Resistors_SMD:R_0805, symbol R
- C1, C2, C4, C5: value C_Small -> 20pF
- C3: value CP_Small -> 10uF
- C6, C7, C8: value C_Small -> 0.1uF
- C9: value C_Small -> 1uF
- R1, R2, R3, R4: value R_Small -> 33 Ohm
- Y1, Y2: value Crystal_Small -> 12MHz
Connections:
- net GND: now also C10.1, C11.2, C12.1, C13.2, R5.2, R6.2
- net Vcc_3.3V: now also C10.2, C11.1, C12.2, C13.1; no longer C6.1
- net ed_VBCOMP: now reaches C9.1, U3.22 (VBCOMP), X1.1 (Vcc), X2.1 (Vcc)
- net RES_ehost: now reaches P2.2 (P2), U2.12 (~RES)
- net ehost_DM: now reaches R2.1, U2.20 (D-)
- net ehost_DP: now reaches R1.1, U2.21 (D+)
- net at U2.4 (GPOUT0): now also D1.2 (A)
- net RES_edevice: now reaches P3.2 (P2), U3.12 (~RES)
- net edevice_DM: now reaches R3.2, U3.20 (D-)
- net edevice_DP: now reaches R4.2, U3.21 (D+)
- net at U3.4 (GPOUT0): now also D2.2 (A)
- net at C3.1, P1.1 (P1), U1.3 (Vin): now also C6.1
- new net: D2.1 (K), R6.1
- new net: D1.1 (K), R5.1
Other:
- moved on the sheet: C3, C6, C9, R1, R2, R3, R4
